File: edge-b/hardware/kicad_sailframes-b1.kicad_pcb (KiCad board)
At the start: 2 copper layers, 0 parts

Commit message: B1 PCB outline v0.4 (Option B) + pin map for capture
PCB outline simplified to small centered rectangle for horizontal-antenna
design path:
- 80 x 56 mm rounded rectangle centered on Polycase ML-34F interior
- R = 10 mm corner fillets (clears 4 corner brass-insert towers laterally
  with ~1.4 mm margin)
- 4 mounting holes NPTH 3.18 mm at the 4 inner Polycase PCB-mounting
  bosses (50 x 28.6 mm pattern)
- No cover-screw clearance through PCB (cover screws engage corner brass
  inserts independently)
- Embedded Polycase template bitmap overlay on Dwgs.User for reference

This replaces v0.3 (asymmetric truncation that didn't match the Polycase
template anywhere and produced a lopsided hole layout). Trade-off
documented: small PCB doesn't host the original 85 x 56 mm TFT module;
B1 boats will use a smaller TFT (arriving 2026-05-19 for fit check).

Antenna will live on a separate carrier PCB perpendicular to main PCB,
panelized at JLCPCB. 50 x 50 mm YFGC007E3A fits in the wider section
of the tapered enclosure interior (53 mm at gasket seat, 49 mm at base
floor).

B1_PIN_MAP.md: complete pin map and net naming reference for schematic
capture. Covers all 5 power rails, every ESP32 GPIO, LC29HEAMD, BNO085,
TFT, microSD, the magnetic toggle latch, and status LEDs. Authoritative
pin numbers for U_FF (SN74LVC1G74DCTR) and U_RST (MAX809T) come from the
JLC2KiCadLib symbols, not the spec's illustrative prose (per spec
checklist line 1267). Includes 10 ERC sanity rules keyed to the spec's
verification checklist.

Polycase_ML-34F_drawing.pdf: official Polycase datasheet, source of
truth for ML-34BF-PCB template dimensions.

Co-Authored-By: Claude Opus 4.7 (1M context) <noreply@anthropic.com>
Other:
- board outline added: 80 x 56 mm
- board text added: "B1 PCB outline v0.4 — Option B: small centered rectangle 80 x 56 mm centered on Polycase interior, R=10 mm corner fillets 4 mounting holes NPTH 3.18 mm at +/-(25, 14.3) mm from Polycase center (inner PCB-mounting boss positions, 50 x 28.6 mm pattern) Clears 4 corner brass-insert towers laterally (no cover-screw holes through PCB) Cover screws engage corner brass inserts independently of PCB Anten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"
